Commit message: update

File: ROS/scara_robot/urdf/scara.urdf (robot description, URDF)
Before this commit: robot scara, 2 links, 1 joints
Links:
- added link link1b; visual cylinder length=0.6 radius=0.3
- link base_link: geometry visual cylinder length=1 radius=0.3
Joints:
- added joint link1_to_link1b: type fixed, parent link1, child link1b, origin xyz=0 0 0.6 rpy=0 0 0

Commit message: update

File: ROS/scara_robot/urdf/scara.urdf (robot description, URDF)
Before this commit: robot scara, 3 links, 2 joints
Links:
- added link link2; visual box size=3 0.6 0.6
- added link link2b; visual cylinder length=0.6 radius=0.3
- added link link2c; visual cylinder length=0.6 radius=0.3
- added link link_ee; visual cylinder length=2 radius=0.1
Joints:
- added joint link1_to_link2b: type fixed, parent link1, child link2b, origin xyz=3 0 0 rpy=0 0 0
- added joint link2_to_link2c: type fixed, parent link2, child link2c, origin xyz=3 0 0 rpy=0 0 0
- added joint link2b_to_link2: type revolute, parent link2b, child link2, origin xyz=0 0 0 rpy=0 0 0, axis 0 0 1, limit lower=-2.5 upper=2.5 effort=1000.0 velocity=0.5
- added joint link2c_to_link_ee: type prismatic, parent link2c, child link_ee, origin xyz=0 0 0 rpy=0 0 0, axis 0 0 1, limit lower=-0.5 upper=0.5 effort=1000.0 velocity=0.5
- joint base_link_to_link1: origin xyz=0 0 0.6 rpy=0 0 0 -> xyz=0 0 1.3 rpy=0 0 0
- joint link1_to_link1b: origin xyz=0 0 0.6 rpy=0 0 0 -> xyz=0 0 0 rpy=0 0 0

Commit message: update

File: ROS/scara_robot/urdf/scara.urdf (robot description, URDF)
Before this commit: robot scara, 7 links, 6 joints
Joints:
- joint base_link_to_link1: type revolute -> continuous
- joint link2c_to_link_ee: limit lower=-0.5 upper=0.5 effort=1000.0 velocity=0.5 -> lower=-1.5 upper=-0.5 effort=1000.0 velocity=0.5
