Commit message: update

File: ROS/scara_robot/urdf/scara.urdf.xacro (robot description, xacro)
@@ -1,4 +1,5 @@
 <?xml version="1.0"?>
-<robot name="scara">
+<robot name="scara" xmlns:xacro="http://ros.org/wiki/xacro">
+<xacro:property name="height" value="1" />
     <!--    define materials-->
     <material name="blue">
@@ -16,5 +17,5 @@
             <origin rpy="0 0 0" xyz="0 0 0.5"/>
             <geometry>
-                <cylinder length="1" radius="0.3"/>
+                <cylinder length="${height}" radius="0.3"/>
             </geometry>
             <material name="green"/>

Commit message: update

File: ROS/scara_robot/urdf/scara.urdf.xacro (robot description, xacro)
@@ -2,4 +2,5 @@
 <robot name="scara" xmlns:xacro="http://ros.org/wiki/xacro">
 <xacro:property name="height" value="1" />
+<xacro:property name="length" value="3" />
     <!--    define materials-->
     <material name="blue">
@@ -37,5 +38,5 @@
             <origin rpy="0 0 0" xyz="1.5 0 0"/>
             <geometry>
-                <box size="3 0.6 0.6"/>
+                <box size="${length} 0.6 0.6"/>
             </geometry>
             <material name="green"/>
@@ -57,5 +58,5 @@
             <origin rpy="0 0 0" xyz="1.5 0 0"/>
             <geometry>
-                <box size="3 0.6 0.6"/>
+                <box size="${length} 0.6 0.6"/>
             </geometry>
             <material name="green"/>

Commit message: update

File: ROS/scara_robot/urdf/scara.urdf.xacro (robot description, xacro)
@@ -1,13 +1,35 @@
 <?xml version="1.0"?>
 <robot name="scara" xmlns:xacro="http://ros.org/wiki/xacro">
-<xacro:property name="height" value="1" />
-<xacro:property name="length" value="3" />
+<!--    <xacro:include filename="$(find scara_robot)/urdf/scara.gazebo"/>-->
+    <xacro:property name="height" value="1"/>
+    <xacro:property name="length" value="3"/>
+    <gazebo reference="base_link">
+        <material>Gazebo/Green</material>
+    </gazebo>
+    <gazebo reference="link1">
+        <material>Gazebo/Green</material>
+    </gazebo>
+    <gazebo reference="link2">
+        <material>Gazebo/Green</material>
+    </gazebo>
+    <gazebo reference="link_ee">
+        <material>Gazebo/Green</material>
+    </gazebo>
+    <gazebo reference="link1b">
+        <material>Gazebo/Blue</material>
+    </gazebo>
+    <gazebo reference="link2b">
+        <material>Gazebo/Blue</material>
+    </gazebo>
+    <gazebo reference="link2c">
+        <material>Gazebo/Blue</material>
+    </gazebo>
     <!--    define materials-->
-    <material name="blue">
-        <color rgba="0 0 0.8 0.5"/>
-    </material>
-    <material name="green">
-        <color rgba="0 1 0 0.5"/>
-    </material>
+    <!--    <material name="blue">-->
+    <!--        <color rgba="0 0 0.8 0.5"/>-->
+    <!--    </material>-->
+    <!--    <material name="green">-->
+    <!--        <color rgba="0 1 0 0.5"/>-->
+    <!--    </material>-->
     <!--    <material name="green">-->
     <!--        <color rgba="1 1 1 1"/>-->
@@ -20,5 +42,5 @@
                 <cylinder length="${height}" radius="0.3"/>
             </geometry>
-            <material name="green"/>
+            <!--            <material name="green"/>-->
         </visual>
     </link>
@@ -30,5 +52,5 @@
                 <cylinder length="0.6" radius="0.3"/>
             </geometry>
-            <material name="blue"/>
+            <!--            <material name="blue"/>-->
         </visual>
     </link>
@@ -40,5 +62,5 @@
                 <box size="${length} 0.6 0.6"/>
             </geometry>
-            <material name="green"/>
+            <!--            <material name="green"/>-->
         </visual>
     </link>
@@ -50,5 +72,5 @@
                 <cylinder length="0.6" radius="0.3"/>
             </geometry>
-            <material name="blue"/>
+            <!--            <material name="blue"/>-->
         </visual>
     </link>
@@ -60,5 +82,5 @@
                 <box size="${length} 0.6 0.6"/>
             </geometry>
-            <material name="green"/>
+            <!--            <material name="green"/>-->
         </visual>
     </link>
@@ -70,5 +92,5 @@
                 <cylinder length="0.6" radius="0.3"/>
             </geometry>
-            <material name="blue"/>
+            <!--            <material name="blue"/>-->
         </visual>
     </link>
@@ -80,5 +102,5 @@
                 <cylinder length="2" radius="0.1"/>
             </geometry>
-            <material name="green"/>
+            <!--            <material name="green"/>-->
         </visual>
     </link>

Commit message: update

File: ROS/scara_robot/urdf/scara.urdf.xacro (robot description, xacro)
@@ -1,38 +1,13 @@
 <?xml version="1.0"?>
 <robot name="scara" xmlns:xacro="http://ros.org/wiki/xacro">
-<!--    <xacro:include filename="$(find scara_robot)/urdf/scara.gazebo"/>-->
     <xacro:property name="height" value="1"/>
     <xacro:property name="length" value="3"/>
-    <gazebo reference="base_link">
-        <material>Gazebo/Green</material>
-    </gazebo>
-    <gazebo reference="link1">
-        <material>Gazebo/Green</material>
-    </gazebo>
-    <gazebo reference="link2">
-        <material>Gazebo/Green</material>
-    </gazebo>
-    <gazebo reference="link_ee">
-        <material>Gazebo/Green</material>
-    </gazebo>
-    <gazebo reference="link1b">
-        <material>Gazebo/Blue</material>
-    </gazebo>
-    <gazebo reference="link2b">
-        <material>Gazebo/Blue</material>
-    </gazebo>
-    <gazebo reference="link2c">
-        <material>Gazebo/Blue</material>
-    </gazebo>
     <!--    define materials-->
-    <!--    <material name="blue">-->
-    <!--        <color rgba="0 0 0.8 0.5"/>-->
-    <!--    </material>-->
-    <!--    <material name="green">-->
-    <!--        <color rgba="0 1 0 0.5"/>-->
-    <!--    </material>-->
-    <!--    <material name="green">-->
-    <!--        <color rgba="1 1 1 1"/>-->
-    <!--    </material>-->
+    <material name="blue">
+        <color rgba="0 0 0.8 0.5"/>
+    </material>
+    <material name="green">
+        <color rgba="0 1 0 0.5"/>
+    </material>
     <!--  base link-->
     <link name="base_link">
@@ -42,5 +17,5 @@
                 <cylinder length="${height}" radius="0.3"/>
             </geometry>
-            <!--            <material name="green"/>-->
+            <material name="green"/>
         </visual>
     </link>
@@ -52,5 +27,5 @@
                 <cylinder length="0.6" radius="0.3"/>
             </geometry>
-            <!--            <material name="blue"/>-->
+            <material name="blue"/>
         </visual>
     </link>
@@ -62,5 +37,5 @@
                 <box size="${length} 0.6 0.6"/>
             </geometry>
-            <!--            <material name="green"/>-->
+            <material name="green"/>
         </visual>
     </link>
@@ -72,5 +47,5 @@
                 <cylinder length="0.6" radius="0.3"/>
             </geometry>
-            <!--            <material name="blue"/>-->
+            <material name="blue"/>
         </visual>
     </link>
@@ -92,5 +67,5 @@
                 <cylinder length="0.6" radius="0.3"/>
             </geometry>
-            <!--            <material name="blue"/>-->
+            <material name="blue"/>
         </visual>
     </link>
@@ -102,5 +77,5 @@
                 <cylinder length="2" radius="0.1"/>
             </geometry>
-            <!--            <material name="green"/>-->
+            <material name="green"/>
         </visual>
     </link>
