Commit message: update

File: ROS/my_fbot/my_fbot/urdf/my_fbot.xacro (robot description, xacro)
@@ -3,8 +3,8 @@
     <xacro:include filename="$(find my_fbot)/urdf/my_fbot.gazebo"/>
     <!--    VARIABLES-->
-    <xacro:property name="chassis_height" value=".2"/>
-    <xacro:property name="chassis_radius" value=".25"/>
+    <xacro:property name="chassis_height" value=".1"/>
+    <xacro:property name="chassis_radius" value=".1"/>
     <xacro:property name="wheel_thickness" value=".05"/>
-    <xacro:property name="wheel_radius" value=".1"/>
+    <xacro:property name="wheel_radius" value=".05"/>
     <!--    MATERIALS-->
     <gazebo reference="chassis">
@@ -26,5 +26,5 @@
     <!--    chassis link-->
     <link name='chassis'>
-        <pose>0 0 0.1 0 0 0</pose>
+        <pose>0 0 0 0 0 0</pose>
         <inertial>
             <mass value="15.0"/>
@@ -37,5 +37,5 @@
         </inertial>
         <collision name='collision'>
-            <origin xyz="0 0 0.05" rpy=" 0 0 0"/>
+            <origin xyz="0 0 ${wheel_radius/2}" rpy=" 0 0 0"/>
             <geometry>
                 <cylinder length="${chassis_height}" radius="${chassis_radius}"/>
@@ -43,5 +43,5 @@
         </collision>
         <visual name='chassis_visual'>
-            <origin xyz="0 0 0.05" rpy=" 0 0 0"/>
+            <origin xyz="0 0 ${wheel_radius/2}" rpy=" 0 0 0"/>
             <geometry>
                 <cylinder length="${chassis_height}" radius="${chassis_radius}"/>
@@ -50,5 +50,5 @@
         <!--        SUPPORT WHEELS-->
         <collision name='back_caster_collision'>
-            <origin xyz="-0.15 0 -0.05" rpy=" 0 0 0"/>
+            <origin xyz="-${chassis_radius/3} 0 -0.025" rpy=" 0 0 0"/>
             <geometry>
                 <sphere radius="${wheel_radius/2}"/>
@@ -56,5 +56,5 @@
         </collision>
         <visual name='back_caster_visual'>
-            <origin xyz="-0.15 0 -0.05" rpy=" 0 0 0"/>
+            <origin xyz="-${chassis_radius/3} 0 -0.025" rpy=" 0 0 0"/>
             <geometry>
                 <sphere radius="${wheel_radius/2}"/>
@@ -62,5 +62,5 @@
         </visual>
         <collision name='front_caster_collision'>
-            <origin xyz="0.15 0 -0.05" rpy=" 0 0 0"/>
+            <origin xyz="${chassis_radius/3} 0 -0.025" rpy=" 0 0 0"/>
             <geometry>
                 <sphere radius="${wheel_radius/2}"/>
@@ -68,5 +68,5 @@
         </collision>
         <visual name='front_caster_visual'>
-            <origin xyz="0.15 0 -0.05" rpy=" 0 0 0"/>
+            <origin xyz="${chassis_radius/3} 0 -0.025" rpy=" 0 0 0"/>
             <geometry>
                 <sphere radius="${wheel_radius/2}"/>
@@ -75,5 +75,5 @@
         <!--        LIDAR SUPPORT-->
         <collision name='lidar_support_collision'>
-            <origin xyz="-0.15 0 ${chassis_height-0.025}" rpy=" 0 0 0"/>
+            <origin xyz="-0.05 0 ${chassis_height-0.02}" rpy=" 0 0 0"/>
             <geometry>
                 <cylinder length="0.05" radius="0.1"/>
@@ -81,7 +81,7 @@
         </collision>
         <visual name='lidar_support_visual'>
-            <origin xyz="-0.15 0 ${chassis_height-0.025}" rpy=" 0 0 0"/>
-            <geometry>
-                <cylinder length="0.05" radius="0.1"/>
+            <origin xyz="-0.05 0 ${chassis_height-0.02}" rpy=" 0 0 0"/>
+            <geometry>
+                <cylinder length="0.02" radius="0.05"/>
             </geometry>
         </visual>
@@ -196,5 +196,5 @@
     </joint>
     <joint name="camera_joint" type="fixed">
-        <origin xyz="0.22 0 ${chassis_height-0.05}" rpy="0 0 0"/>
+        <origin xyz="0.05 0 ${chassis_height-0.02}" rpy="0 0 0"/>
         <parent link="chassis"/>
         <child link="camera"/>
@@ -202,5 +202,5 @@
     </joint>
     <joint name="hokuyo_joint" type="fixed">
-        <origin xyz="-0.15 0 ${chassis_height}" rpy="0 0 0"/>
+        <origin xyz="-0.05 0 ${chassis_height+0.02}" rpy="0 0 0"/>
         <parent link="chassis"/>
         <child link="hokuyo"/>

Commit message: update

File: ROS/my_fbot/my_fbot/urdf/my_fbot.xacro (robot description, xacro)
@@ -196,5 +196,5 @@
     </joint>
     <joint name="camera_joint" type="fixed">
-        <origin xyz="0.05 0 ${chassis_height-0.02}" rpy="0 0 0"/>
+        <origin xyz="0.07 0 ${chassis_height-0.02}" rpy="0 0 0"/>
         <parent link="chassis"/>
         <child link="camera"/>

Commit message: update

File: ROS/my_fbot/my_fbot/urdf/my_fbot.xacro (robot description, xacro)
@@ -5,5 +5,6 @@
     <xacro:property name="chassis_height" value=".1"/>
     <xacro:property name="chassis_radius" value=".1"/>
-    <xacro:property name="wheel_thickness" value=".05"/>
+    <xacro:property name="sup_wheels_height" value="-0.0249"/>
+    <xacro:property name="wheel_thickness" value=".025"/>
     <xacro:property name="wheel_radius" value=".05"/>
     <!--    MATERIALS-->
@@ -50,5 +51,5 @@
         <!--        SUPPORT WHEELS-->
         <collision name='back_caster_collision'>
-            <origin xyz="-${chassis_radius/3} 0 -0.025" rpy=" 0 0 0"/>
+            <origin xyz="-${chassis_radius/3} 0 ${sup_wheels_height}" rpy=" 0 0 0"/>
             <geometry>
                 <sphere radius="${wheel_radius/2}"/>
@@ -56,5 +57,5 @@
         </collision>
         <visual name='back_caster_visual'>
-            <origin xyz="-${chassis_radius/3} 0 -0.025" rpy=" 0 0 0"/>
+            <origin xyz="-${chassis_radius/3} 0 ${sup_wheels_height}" rpy=" 0 0 0"/>
             <geometry>
                 <sphere radius="${wheel_radius/2}"/>
@@ -62,5 +63,5 @@
         </visual>
         <collision name='front_caster_collision'>
-            <origin xyz="${chassis_radius/3} 0 -0.025" rpy=" 0 0 0"/>
+            <origin xyz="${chassis_radius/3} 0 ${sup_wheels_height}" rpy=" 0 0 0"/>
             <geometry>
                 <sphere radius="${wheel_radius/2}"/>
@@ -68,5 +69,5 @@
         </collision>
         <visual name='front_caster_visual'>
-            <origin xyz="${chassis_radius/3} 0 -0.025" rpy=" 0 0 0"/>
+            <origin xyz="${chassis_radius/3} 0 ${sup_wheels_height}" rpy=" 0 0 0"/>
             <geometry>
                 <sphere radius="${wheel_radius/2}"/>

Commit message: update

File: ROS/my_fbot/my_fbot/urdf/my_fbot.xacro (robot description, xacro)
@@ -196,10 +196,19 @@
         <dynamics damping="1.0" friction="1.0"/>
     </joint>
-    <joint name="camera_joint" type="fixed">
-        <origin xyz="0.07 0 ${chassis_height-0.02}" rpy="0 0 0"/>
+    <joint name="camera_joint" type="continuous">
+        <axis xyz="0 1 1"/>
+        <origin xyz="0.09 0 ${chassis_height-0.1}" rpy="0 0 0"/>
         <parent link="chassis"/>
         <child link="camera"/>
-        <axis xyz="0 1 0"/>
-    </joint>
+    </joint>
+    <transmission name="camera_transmission">
+        <type>transmission_interface/SimpleTransmission</type>
+        <actuator name="$camera_motor">
+            <mechanicalReduction>1</mechanicalReduction>
+        </actuator>
+        <joint name="camera_joint">
+            <hardwareInterface>hardware_interface/PositionJointInterface</hardwareInterface>
+        </joint>
+    </transmission>
     <joint name="hokuyo_joint" type="fixed">
         <origin xyz="-0.05 0 ${chassis_height+0.02}" rpy="0 0 0"/>

Commit message: update

File: ROS/my_fbot/my_fbot/urdf/my_fbot.xacro (robot description, xacro)
@@ -139,9 +139,9 @@
         <inertial>
             <mass value="0.1"/>
-            <origin xyz="0 0 0" rpy="0 0 0"/>
+            <origin xyz="0 0 0" rpy="0 0.01 0"/>
             <inertia ixx="0.03" ixy="0.0" ixz="0.0" iyy="0.03" iyz="0.0" izz="0.03"/>
         </inertial>
         <collision>
-            <origin xyz="0 0 0" rpy="0 0 0"/>
+            <origin xyz="0 0 0" rpy="0 0.01 0"/>
             <geometry>
                 <sphere radius="0.02"/>
@@ -149,5 +149,5 @@
         </collision>
         <visual>
-            <origin xyz="0 0 0" rpy="0 0 0"/>
+            <origin xyz="0 0 0" rpy="0 0.01 0"/>
             <geometry>
                 <mesh filename="package://computer_vision_pkg/meshes/head.dae" scale=".5 .5 .5"/>

Commit message: update

File: ROS/my_fbot/my_fbot/urdf/my_fbot.xacro (robot description, xacro)
@@ -139,9 +139,9 @@
         <inertial>
             <mass value="0.1"/>
-            <origin xyz="0 0 0" rpy="0 0.01 0"/>
+            <origin xyz="0 0 0" rpy="0 0 0"/>
             <inertia ixx="0.03" ixy="0.0" ixz="0.0" iyy="0.03" iyz="0.0" izz="0.03"/>
         </inertial>
         <collision>
-            <origin xyz="0 0 0" rpy="0 0.01 0"/>
+            <origin xyz="0 0 0" rpy="0 0 0"/>
             <geometry>
                 <sphere radius="0.02"/>
@@ -149,5 +149,5 @@
         </collision>
         <visual>
-            <origin xyz="0 0 0" rpy="0 0.01 0"/>
+            <origin xyz="0 0 0" rpy="0 0 0"/>
             <geometry>
                 <mesh filename="package://computer_vision_pkg/meshes/head.dae" scale=".5 .5 .5"/>
@@ -198,17 +198,17 @@
     <joint name="camera_joint" type="continuous">
         <axis xyz="0 1 1"/>
-        <origin xyz="0.09 0 ${chassis_height-0.1}" rpy="0 0 0"/>
+        <origin xyz="0.09 0 ${chassis_height-0.1}" rpy="0 0.2 0"/>
         <parent link="chassis"/>
         <child link="camera"/>
     </joint>
-    <transmission name="camera_transmission">
-        <type>transmission_interface/SimpleTransmission</type>
-        <actuator name="$camera_motor">
-            <mechanicalReduction>1</mechanicalReduction>
-        </actuator>
-        <joint name="camera_joint">
-            <hardwareInterface>hardware_interface/PositionJointInterface</hardwareInterface>
-        </joint>
-    </transmission>
+    <!--    <transmission name="camera_transmission">-->
+    <!--        <type>transmission_interface/SimpleTransmission</type>-->
+    <!--        <actuator name="$camera_motor">-->
+    <!--            <mechanicalReduction>1</mechanicalReduction>-->
+    <!--        </actuator>-->
+    <!--        <joint name="camera_joint">-->
+    <!--            <hardwareInterface>hardware_interface/PositionJointInterface</hardwareInterface>-->
+    <!--        </joint>-->
+    <!--    </transmission>-->
     <joint name="hokuyo_joint" type="fixed">
         <origin xyz="-0.05 0 ${chassis_height+0.02}" rpy="0 0 0"/>

Commit message: update

File: ROS/my_fbot/my_fbot/urdf/my_fbot.xacro (robot description, xacro)
@@ -198,17 +198,17 @@
     <joint name="camera_joint" type="continuous">
         <axis xyz="0 1 1"/>
-        <origin xyz="0.09 0 ${chassis_height-0.1}" rpy="0 0.2 0"/>
+        <origin xyz="0.09 0 ${chassis_height-0.1}" rpy="0 0 0"/>
         <parent link="chassis"/>
         <child link="camera"/>
     </joint>
-    <!--    <transmission name="camera_transmission">-->
-    <!--        <type>transmission_interface/SimpleTransmission</type>-->
-    <!--        <actuator name="$camera_motor">-->
-    <!--            <mechanicalReduction>1</mechanicalReduction>-->
-    <!--        </actuator>-->
-    <!--        <joint name="camera_joint">-->
-    <!--            <hardwareInterface>hardware_interface/PositionJointInterface</hardwareInterface>-->
-    <!--        </joint>-->
-    <!--    </transmission>-->
+        <transmission name="camera_transmission">
+            <type>transmission_interface/SimpleTransmission</type>
+            <actuator name="$camera_motor">
+                <mechanicalReduction>1</mechanicalReduction>
+            </actuator>
+            <joint name="camera_joint">
+                <hardwareInterface>hardware_interface/PositionJointInterface</hardwareInterface>
+            </joint>
+        </transmission>
     <joint name="hokuyo_joint" type="fixed">
         <origin xyz="-0.05 0 ${chassis_height+0.02}" rpy="0 0 0"/>

Commit message: update

File: ROS/my_fbot/my_fbot/urdf/my_fbot.xacro (robot description, xacro)
@@ -151,5 +151,5 @@
             <origin xyz="0 0 0" rpy="0 0 0"/>
             <geometry>
-                <mesh filename="package://computer_vision_pkg/meshes/head.dae" scale=".5 .5 .5"/>
+                <mesh filename="package://my_fbot/meshes/head.dae" scale=".5 .5 .5"/>
             </geometry>
         </visual>
