Commit message: update

File: ROS/p_jfernandes/urdf/p_jfernandes.gazebo.xacro (robot description, xacro)
@@ -5,14 +5,15 @@
     <xacro:arg name="imu_visual" default="false"/>
     <xacro:arg name="main_color" default="Blue"/>
-    <gazebo reference="base_link">
+    <xacro:property name="robot_name" value="p_jfernandes/"/>
+    <gazebo reference="${robot_name}base_link">
         <material>Gazebo/$(arg main_color)</material>
     </gazebo>
-    <gazebo reference="stem">
+    <gazebo reference="${robot_name}stem">
         <material>Gazebo/$(arg main_color)</material>
     </gazebo>
-    <gazebo reference="top">
+    <gazebo reference="${robot_name}top">
         <material>Gazebo/$(arg main_color)</material>
     </gazebo>
-    <gazebo reference="wheel_left_link">
+    <gazebo reference="${robot_name}wheel_left_link">
         <mu1>0.1</mu1>
         <mu2>0.1</mu2>
@@ -24,5 +25,5 @@
         <material>Gazebo/$(arg main_color)</material>
     </gazebo>
-    <gazebo reference="wheel_right_link">
+    <gazebo reference="${robot_name}wheel_right_link">
         <mu1>0.1</mu1>
         <mu2>0.1</mu2>
@@ -34,5 +35,5 @@
         <material>Gazebo/$(arg main_color)</material>
     </gazebo>
-    <gazebo reference="caster_back_right_link">
+    <gazebo reference="${robot_name}caster_back_right_link">
         <mu1>0.1</mu1>
         <mu2>0.1</mu2>
@@ -43,5 +44,5 @@
         <material>Gazebo/$(arg main_color)</material>
     </gazebo>
-    <gazebo reference="caster_back_left_link">
+    <gazebo reference="${robot_name}caster_back_left_link">
         <mu1>0.1</mu1>
         <mu2>0.1</mu2>
@@ -52,5 +53,5 @@
         <material>Gazebo/$(arg main_color)</material>
     </gazebo>
-    <gazebo reference="imu_link">
+    <gazebo reference="${robot_name}imu_link">
         <sensor type="imu" name="imu">
             <always_on>true</always_on>
@@ -61,10 +62,10 @@
     <gazebo>
         <plugin name="turtlebot3_waffle_pi_controller" filename="libgazebo_ros_diff_drive.so">
-            <commandTopic>p_jfernandes/cmd_vel</commandTopic>
+            <commandTopic>${robot_name}cmd_vel</commandTopic>
             <odometryTopic>odom</odometryTopic>
-            <odometryFrame>odom</odometryFrame>
+            <odometryFrame>${robot_name}odom</odometryFrame>
             <odometrySource>world</odometrySource>
             <publishOdomTF>true</publishOdomTF>
-            <robotBaseFrame>base_footprint</robotBaseFrame>
+            <robotBaseFrame>${robot_name}base_footprint</robotBaseFrame>
             <publishWheelTF>false</publishWheelTF>
             <publishTf>true</publishTf>
@@ -85,8 +86,8 @@
         <plugin name="imu_plugin" filename="libgazebo_ros_imu.so">
             <alwaysOn>true</alwaysOn>
-            <bodyName>imu_link</bodyName>
-            <frameName>imu_link</frameName>
-            <topicName>p_jfernandes/imu</topicName>
-            <serviceName>p_jfernandes/imu_service</serviceName>
+            <bodyName>${robot_name}imu_link</bodyName>
+            <frameName>${robot_name}imu_link</frameName>
+            <topicName>${robot_name}imu</topicName>
+            <serviceName>${robot_name}imu_service</serviceName>
             <gaussianNoise>0.0</gaussianNoise>
             <updateRate>0</updateRate>
@@ -110,5 +111,5 @@
         </plugin>
     </gazebo>
-    <gazebo reference="base_scan">
+    <gazebo reference="${robot_name}base_scan">
         <material>Gazebo/FlatBlack</material>
         <sensor type="ray" name="lds_lfcd_sensor">
@@ -137,11 +138,11 @@
             </ray>
             <plugin name="gazebo_ros_lds_lfcd_controller" filename="libgazebo_ros_laser.so">
-                <topicName>p_jfernandes/scan</topicName>
-                <frameName>base_scan</frameName>
+                <topicName>${robot_name}scan</topicName>
+                <frameName>${robot_name}base_scan</frameName>
             </plugin>
         </sensor>
     </gazebo>
     <!--link : https://www.raspberrypi.org/documentation/hardware/camera/-->
-    <gazebo reference="camera_rgb_frame">
+    <gazebo reference="${robot_name}camera_rgb_frame">
         <sensor type="camera" name="Pi Camera">
             <always_on>true</always_on>
@@ -164,6 +165,6 @@
                 <alwaysOn>true</alwaysOn>
                 <updateRate>30.0</updateRate>
-                <cameraName>p_jfernandes/camera</cameraName>
-                <frameName>camera_rgb_optical_frame</frameName>
+                <cameraName>${robot_name}camera</cameraName>
+                <frameName>${robot_name}camera_rgb_optical_frame</frameName>
                 <imageTopicName>rgb/image_raw</imageTopicName>
                 <cameraInfoTopicName>rgb/camera_info</cameraInfoTopicName>
