Commit message: update

File: ROS/green_turtlebot3/urdf/green_turtlebot3.gazebo.xacro (robot description, xacro)
@@ -1,7 +1,9 @@
 <?xml version="1.0"?>
-<robot name="p_jfernandes_sim" xmlns:xacro="http://ros.org/wiki/xacro">
+<robot name="green_turtlebot3_sim" xmlns:xacro="http://ros.org/wiki/xacro">
     <xacro:arg name="laser_visual" default="false"/>
     <xacro:arg name="camera_visual" default="false"/>
     <xacro:arg name="imu_visual" default="false"/>
+    <!--    robot main color-->
+    <xacro:arg name="main_color" default="Green"/>
     <gazebo reference="base_link">
         <material>Gazebo/DarkGrey</material>
@@ -11,5 +13,5 @@
     </gazebo>
     <gazebo reference="top">
-        <material>Gazebo/Blue</material>
+        <material>Gazebo/$(arg main_color)</material>
     </gazebo>
     <gazebo reference="wheel_left_link">
@@ -21,5 +23,5 @@
         <maxVel>0.1</maxVel>
         <fdir1>1 0 0</fdir1>
-        <material>Gazebo/Blue</material>
+        <material>Gazebo/$(arg main_color)</material>
     </gazebo>
     <gazebo reference="wheel_right_link">
@@ -31,5 +33,5 @@
         <maxVel>0.1</maxVel>
         <fdir1>1 0 0</fdir1>
-        <material>Gazebo/Blue</material>
+        <material>Gazebo/$(arg main_color)</material>
     </gazebo>
     <gazebo reference="caster_back_right_link">
@@ -60,5 +62,5 @@
     <gazebo>
         <plugin name="turtlebot3_waffle_pi_controller" filename="libgazebo_ros_diff_drive.so">
-            <commandTopic>p_jfernandes/cmd_vel</commandTopic>
+            <commandTopic>green_turtlebot3/cmd_vel</commandTopic>
             <odometryTopic>odom</odometryTopic>
             <odometryFrame>odom</odometryFrame>
@@ -86,6 +88,6 @@
             <bodyName>imu_link</bodyName>
             <frameName>imu_link</frameName>
-            <topicName>p_jfernandes/imu</topicName>
-            <serviceName>p_jfernandes/imu_service</serviceName>
+            <topicName>green_turtlebot3/imu</topicName>
+            <serviceName>green_turtlebot3/imu_service</serviceName>
             <gaussianNoise>0.0</gaussianNoise>
             <updateRate>0</updateRate>
@@ -136,5 +138,5 @@
             </ray>
             <plugin name="gazebo_ros_lds_lfcd_controller" filename="libgazebo_ros_laser.so">
-                <topicName>p_jfernandes/scan</topicName>
+                <topicName>green_turtlebot3/scan</topicName>
                 <frameName>base_scan</frameName>
             </plugin>
@@ -151,5 +153,5 @@
                     <!--                    <width>640</width>-->
                     <!--                    <height>480</height>-->
-                    <width>1000</width>
+                    <width>1200</width>
                     <height>800</height>
                     <format>R8G8B8</format>
@@ -163,5 +165,5 @@
                 <alwaysOn>true</alwaysOn>
                 <updateRate>30.0</updateRate>
-                <cameraName>p_jfernandes/camera</cameraName>
+                <cameraName>green_turtlebot3/camera</cameraName>
                 <frameName>camera_rgb_optical_frame</frameName>
                 <imageTopicName>rgb/image_raw</imageTopicName>

File: ROS/red_turtlebot3/urdf/red_turtlebot3.gazebo.xacro (robot description, xacro)
@@ -4,4 +4,5 @@
     <xacro:arg name="camera_visual" default="false"/>
     <xacro:arg name="imu_visual" default="false"/>
+    <xacro:arg name="main_color" default="Red"/>
     <gazebo reference="base_link">
         <material>Gazebo/DarkGrey</material>
@@ -11,5 +12,5 @@
     </gazebo>
     <gazebo reference="top">
-        <material>Gazebo/Red</material>
+        <material>Gazebo/$(arg main_color)</material>
     </gazebo>
     <gazebo reference="wheel_left_link">
@@ -21,5 +22,5 @@
         <maxVel>0.1</maxVel>
         <fdir1>1 0 0</fdir1>
-        <material>Gazebo/Blue</material>
+        <material>Gazebo/$(arg main_color)</material>
     </gazebo>
     <gazebo reference="wheel_right_link">
@@ -31,5 +32,5 @@
         <maxVel>0.1</maxVel>
         <fdir1>1 0 0</fdir1>
-        <material>Gazebo/Blue</material>
+        <material>Gazebo/$(arg main_color)</material>
     </gazebo>
     <gazebo reference="caster_back_right_link">
@@ -87,5 +88,5 @@
             <frameName>imu_link</frameName>
             <topicName>red_turtlebot3/imu</topicName>
-            <serviceName>imu_service</serviceName>
+            <serviceName>red_turtlebot3/imu_service</serviceName>
             <gaussianNoise>0.0</gaussianNoise>
             <updateRate>0</updateRate>

Commit message: update

File: ROS/green_turtlebot3/urdf/green_turtlebot3.gazebo.xacro (robot description, xacro)
@@ -7,8 +7,8 @@
     <xacro:arg name="main_color" default="Green"/>
     <gazebo reference="base_link">
-        <material>Gazebo/DarkGrey</material>
+        <material>Gazebo/$(arg main_color)</material>
     </gazebo>
     <gazebo reference="stem">
-        <material>Gazebo/DarkGrey</material>
+        <material>Gazebo/$(arg main_color)</material>
     </gazebo>
     <gazebo reference="top">
@@ -42,5 +42,5 @@
         <minDepth>0.001</minDepth>
         <maxVel>1.0</maxVel>
-        <material>Gazebo/Blue</material>
+        <material>Gazebo/$(arg main_color)</material>
     </gazebo>
     <gazebo reference="caster_back_left_link">
@@ -51,5 +51,5 @@
         <minDepth>0.001</minDepth>
         <maxVel>1.0</maxVel>
-        <material>Gazebo/Blue</material>
+        <material>Gazebo/$(arg main_color)</material>
     </gazebo>
     <gazebo reference="imu_link">

File: ROS/p_jfernandes/urdf/p_jfernandes.gazebo.xacro (robot description, xacro)
@@ -4,12 +4,13 @@
     <xacro:arg name="camera_visual" default="false"/>
     <xacro:arg name="imu_visual" default="false"/>
+    <xacro:arg name="main_color" default="Blue"/>
     <gazebo reference="base_link">
-        <material>Gazebo/DarkGrey</material>
+        <material>Gazebo/$(arg main_color)</material>
     </gazebo>
     <gazebo reference="stem">
-        <material>Gazebo/DarkGrey</material>
+        <material>Gazebo/$(arg main_color)</material>
     </gazebo>
     <gazebo reference="top">
-        <material>Gazebo/Blue</material>
+        <material>Gazebo/$(arg main_color)</material>
     </gazebo>
     <gazebo reference="wheel_left_link">
@@ -21,5 +22,5 @@
         <maxVel>0.1</maxVel>
         <fdir1>1 0 0</fdir1>
-        <material>Gazebo/Blue</material>
+        <material>Gazebo/$(arg main_color)</material>
     </gazebo>
     <gazebo reference="wheel_right_link">
@@ -31,5 +32,5 @@
         <maxVel>0.1</maxVel>
         <fdir1>1 0 0</fdir1>
-        <material>Gazebo/Blue</material>
+        <material>Gazebo/$(arg main_color)</material>
     </gazebo>
     <gazebo reference="caster_back_right_link">
@@ -40,5 +41,5 @@
         <minDepth>0.001</minDepth>
         <maxVel>1.0</maxVel>
-        <material>Gazebo/Blue</material>
+        <material>Gazebo/$(arg main_color)</material>
     </gazebo>
     <gazebo reference="caster_back_left_link">
@@ -49,5 +50,5 @@
         <minDepth>0.001</minDepth>
         <maxVel>1.0</maxVel>
-        <material>Gazebo/Blue</material>
+        <material>Gazebo/$(arg main_color)</material>
     </gazebo>
     <gazebo reference="imu_link">

File: ROS/p_jfernandes/urdf/p_jfernandes.urdf.xacro (robot description, xacro)
@@ -4,11 +4,12 @@
     <xacro:include filename="$(find p_jfernandes)/urdf/p_jfernandes.gazebo.xacro"/>
     <xacro:property name="top_length" value="0.03"/>
-    <link name="base_footprint"/>
+    <xacro:property name="robot_name" value="p_jfernandes/"/>
+    <link name="${robot_name}base_footprint"/>
     <joint name="base_joint" type="fixed">
-        <parent link="base_footprint"/>
-        <child link="base_link"/>
+        <parent link="${robot_name}base_footprint"/>
+        <child link="${robot_name}base_link"/>
         <origin xyz="0 0 0.010" rpy="0 0 0"/>
     </joint>
-    <link name="base_link">
+    <link name="${robot_name}base_link">
         <visual>
             <origin xyz="-0.064 0 0.0" rpy="0 0 0"/>
@@ -34,5 +35,5 @@
     </link>
     <!--    add blue element   ********************** -->
-    <link name="stem">
+    <link name="${robot_name}stem">
         <visual>
             <origin xyz="0 0 0.0" rpy="0 0 0"/>
@@ -50,9 +51,9 @@
     </link>
     <joint name="stem_joint" type="fixed">
-        <parent link="base_link"/>
-        <child link="stem"/>
+        <parent link="${robot_name}base_link"/>
+        <child link="${robot_name}stem"/>
         <origin xyz="-0.16 0.07 0.14" rpy="0 0 0"/>
     </joint>
-    <link name="top">
+    <link name="${robot_name}top">
         <visual>
             <origin xyz="0 0 0.0" rpy="0 0 0"/>
@@ -70,16 +71,16 @@
     </link>
     <joint name="top_joint" type="fixed">
-        <parent link="base_link"/>
-        <child link="top"/>
+        <parent link="${robot_name}base_link"/>
+        <child link="${robot_name}top"/>
         <origin xyz="-0.16 0.07 0.19" rpy="0 0 0"/>
     </joint>
     <!--    ************************************************-->
     <joint name="wheel_left_joint" type="continuous">
-        <parent link="base_link"/>
-        <child link="wheel_left_link"/>
+        <parent link="${robot_name}base_link"/>
+        <child link="${robot_name}wheel_left_link"/>
         <origin xyz="0.0 0.144 0.023" rpy="-1.57 0 0"/>
         <axis xyz="0 0 1"/>
     </joint>
-    <link name="wheel_left_link">
+    <link name="${robot_name}wheel_left_link">
         <visual>
             <origin xyz="0 0 0" rpy="1.57 0 0"/>
@@ -105,10 +106,10 @@
     </link>
     <joint name="wheel_right_joint" type="continuous">
-        <parent link="base_link"/>
-        <child link="wheel_right_link"/>
+        <parent link="${robot_name}base_link"/>
+        <child link="${robot_name}wheel_right_link"/>
         <origin xyz="0.0 -0.144 0.023" rpy="-1.57 0 0"/>
         <axis xyz="0 0 1"/>
     </joint>
-    <link name="wheel_right_link">
+    <link name="${robot_name}wheel_right_link">
         <visual>
             <origin xyz="0 0 0" rpy="1.57 0 0"/>
@@ -134,9 +135,9 @@
     </link>
     <joint name="caster_back_right_joint" type="fixed">
-        <parent link="base_link"/>
-        <child link="caster_back_right_link"/>
+        <parent link="${robot_name}base_link"/>
+        <child link="${robot_name}caster_back_right_link"/>
         <origin xyz="-0.177 -0.064 -0.004" rpy="-1.57 0 0"/>
     </joint>
-    <link name="caster_back_right_link">
+    <link name="${robot_name}caster_back_right_link">
         <collision>
             <origin xyz="0 0.001 0" rpy="0 0 0"/>
@@ -154,9 +155,9 @@
     </link>
     <joint name="caster_back_left_joint" type="fixed">
-        <parent link="base_link"/>
-        <child link="caster_back_left_link"/>
+        <parent link="${robot_name}base_link"/>
+        <child link="${robot_name}caster_back_left_link"/>
         <origin xyz="-0.177 0.064 -0.004" rpy="-1.57 0 0"/>
     </joint>
-    <link name="caster_back_left_link">
+    <link name="${robot_name}caster_back_left_link">
         <collision>
             <origin xyz="0 0.001 0" rpy="0 0 0"/>
@@ -174,15 +175,15 @@
     </link>
     <joint name="imu_joint" type="fixed">
-        <parent link="base_link"/>
-        <child link="imu_link"/>
+        <parent link="${robot_name}base_link"/>
+        <child link="${robot_name}imu_link"/>
         <origin xyz="0.0 0 0.068" rpy="0 0 0"/>
     </joint>
-    <link name="imu_link"/>
+    <link name="${robot_name}imu_link"/>
     <joint name="scan_joint" type="fixed">
-        <parent link="base_link"/>
-        <child link="base_scan"/>
+        <parent link="${robot_name}base_link"/>
+        <child link="${robot_name}base_scan"/>
         <origin xyz="-0.064 0 0.122" rpy="0 0 0"/>
     </joint>
-    <link name="base_scan">
+    <link name="${robot_name}base_scan">
         <visual>
             <origin xyz="0 0 0.0" rpy="0 0 0"/>
@@ -208,8 +209,8 @@
     <joint name="camera_joint" type="fixed">
         <origin xyz="0.073 -0.011 0.084" rpy="0 0 0"/>
-        <parent link="base_link"/>
-        <child link="camera_link"/>
-    </joint>
-    <link name="camera_link">
+        <parent link="${robot_name}base_link"/>
+        <child link="${robot_name}camera_link"/>
+    </joint>
+    <link name="${robot_name}camera_link">
         <collision>
             <origin xyz="0.005 0.011 0.013" rpy="0 0 0"/>
@@ -221,13 +222,13 @@
     <joint name="camera_rgb_joint" type="fixed">
         <origin xyz="0.003 0.011 0.009" rpy="0 0 0"/>
-        <parent link="camera_link"/>
-        <child link="camera_rgb_frame"/>
-    </joint>
-    <link name="camera_rgb_frame"/>
+        <parent link="${robot_name}camera_link"/>
+        <child link="${robot_name}camera_rgb_frame"/>
+    </joint>
+    <link name="${robot_name}camera_rgb_frame"/>
     <joint name="camera_rgb_optical_joint" type="fixed">
         <origin xyz="0 0 0" rpy="-1.57 0 -1.57"/>
-        <parent link="camera_rgb_frame"/>
-        <child link="camera_rgb_optical_frame"/>
-    </joint>
-    <link name="camera_rgb_optical_frame"/>
+        <parent link="${robot_name}camera_rgb_frame"/>
+        <child link="${robot_name}camera_rgb_optical_frame"/>
+    </joint>
+    <link name="${robot_name}camera_rgb_optical_frame"/>
 </robot>

File: ROS/red_turtlebot3/urdf/red_turtlebot3.gazebo.xacro (robot description, xacro)
@@ -6,8 +6,8 @@
     <xacro:arg name="main_color" default="Red"/>
     <gazebo reference="base_link">
-        <material>Gazebo/DarkGrey</material>
+        <material>Gazebo/$(arg main_color)</material>
     </gazebo>
     <gazebo reference="stem">
-        <material>Gazebo/DarkGrey</material>
+        <material>Gazebo/$(arg main_color)</material>
     </gazebo>
     <gazebo reference="top">
@@ -41,5 +41,5 @@
         <minDepth>0.001</minDepth>
         <maxVel>1.0</maxVel>
-        <material>Gazebo/Blue</material>
+        <material>Gazebo/$(arg main_color)</material>
     </gazebo>
     <gazebo reference="caster_back_left_link">
@@ -50,5 +50,5 @@
         <minDepth>0.001</minDepth>
         <maxVel>1.0</maxVel>
-        <material>Gazebo/Blue</material>
+        <material>Gazebo/$(arg main_color)</material>
     </gazebo>
     <gazebo reference="imu_link">
