Commit message: update

File: ROS/green_turtlebot3/urdf/green_turtlebot3.gazebo.xacro (robot description, xacro)
@@ -6,14 +6,15 @@
     <!--    robot main color-->
     <xacro:arg name="main_color" default="Green"/>
-    <gazebo reference="base_link">
+    <xacro:property name="robot_name" value="green/"/>
+    <gazebo reference="${robot_name}base_link">
         <material>Gazebo/$(arg main_color)</material>
     </gazebo>
-    <gazebo reference="stem">
-        <material>Gazebo/$(arg main_color)</material>
-    </gazebo>
-    <gazebo reference="top">
-        <material>Gazebo/$(arg main_color)</material>
-    </gazebo>
-    <gazebo reference="wheel_left_link">
+    <!--    <gazebo reference="${robot_name}stem">-->
+    <!--        <material>Gazebo/$(arg main_color)</material>-->
+    <!--    </gazebo>-->
+    <!--    <gazebo reference="${robot_name}top">-->
+    <!--        <material>Gazebo/$(arg main_color)</material>-->
+    <!--    </gazebo>-->
+    <gazebo reference="${robot_name}wheel_left_link">
         <mu1>0.1</mu1>
         <mu2>0.1</mu2>
@@ -25,5 +26,5 @@
         <material>Gazebo/$(arg main_color)</material>
     </gazebo>
-    <gazebo reference="wheel_right_link">
+    <gazebo reference="${robot_name}wheel_right_link">
         <mu1>0.1</mu1>
         <mu2>0.1</mu2>
@@ -35,5 +36,5 @@
         <material>Gazebo/$(arg main_color)</material>
     </gazebo>
-    <gazebo reference="caster_back_right_link">
+    <gazebo reference="${robot_name}caster_back_right_link">
         <mu1>0.1</mu1>
         <mu2>0.1</mu2>
@@ -44,5 +45,5 @@
         <material>Gazebo/$(arg main_color)</material>
     </gazebo>
-    <gazebo reference="caster_back_left_link">
+    <gazebo reference="${robot_name}caster_back_left_link">
         <mu1>0.1</mu1>
         <mu2>0.1</mu2>
@@ -53,5 +54,5 @@
         <material>Gazebo/$(arg main_color)</material>
     </gazebo>
-    <gazebo reference="imu_link">
+    <gazebo reference="${robot_name}imu_link">
         <sensor type="imu" name="imu">
             <always_on>true</always_on>
@@ -62,10 +63,10 @@
     <gazebo>
         <plugin name="turtlebot3_waffle_pi_controller" filename="libgazebo_ros_diff_drive.so">
-            <commandTopic>green_turtlebot3/cmd_vel</commandTopic>
+            <commandTopic>${robot_name}cmd_vel</commandTopic>
             <odometryTopic>odom</odometryTopic>
-            <odometryFrame>odom</odometryFrame>
+            <odometryFrame>${robot_name}odom</odometryFrame>
             <odometrySource>world</odometrySource>
             <publishOdomTF>true</publishOdomTF>
-            <robotBaseFrame>base_footprint</robotBaseFrame>
+            <robotBaseFrame>${robot_name}base_footprint</robotBaseFrame>
             <publishWheelTF>false</publishWheelTF>
             <publishTf>true</publishTf>
@@ -86,8 +87,8 @@
         <plugin name="imu_plugin" filename="libgazebo_ros_imu.so">
             <alwaysOn>true</alwaysOn>
-            <bodyName>imu_link</bodyName>
-            <frameName>imu_link</frameName>
-            <topicName>green_turtlebot3/imu</topicName>
-            <serviceName>green_turtlebot3/imu_service</serviceName>
+            <bodyName>${robot_name}imu_link</bodyName>
+            <frameName>${robot_name}imu_link</frameName>
+            <topicName>${robot_name}imu</topicName>
+            <serviceName>${robot_name}imu_service</serviceName>
             <gaussianNoise>0.0</gaussianNoise>
             <updateRate>0</updateRate>
@@ -111,5 +112,5 @@
         </plugin>
     </gazebo>
-    <gazebo reference="base_scan">
+    <gazebo reference="${robot_name}base_scan">
         <material>Gazebo/FlatBlack</material>
         <sensor type="ray" name="lds_lfcd_sensor">
@@ -138,11 +139,11 @@
             </ray>
             <plugin name="gazebo_ros_lds_lfcd_controller" filename="libgazebo_ros_laser.so">
-                <topicName>green_turtlebot3/scan</topicName>
-                <frameName>base_scan</frameName>
+                <topicName>${robot_name}scan</topicName>
+                <frameName>${robot_name}base_scan</frameName>
             </plugin>
         </sensor>
     </gazebo>
     <!--link : https://www.raspberrypi.org/documentation/hardware/camera/-->
-    <gazebo reference="camera_rgb_frame">
+    <gazebo reference="${robot_name}camera_rgb_frame">
         <sensor type="camera" name="Pi Camera">
             <always_on>true</always_on>
@@ -153,5 +154,5 @@
                     <!--                    <width>640</width>-->
                     <!--                    <height>480</height>-->
-                    <width>1200</width>
+                    <width>1000</width>
                     <height>800</height>
                     <format>R8G8B8</format>
@@ -165,6 +166,6 @@
                 <alwaysOn>true</alwaysOn>
                 <updateRate>30.0</updateRate>
-                <cameraName>green_turtlebot3/camera</cameraName>
-                <frameName>camera_rgb_optical_frame</frameName>
+                <cameraName>${robot_name}camera</cameraName>
+                <frameName>${robot_name}camera_rgb_optical_frame</frameName>
                 <imageTopicName>rgb/image_raw</imageTopicName>
                 <cameraInfoTopicName>rgb/camera_info</cameraInfoTopicName>

File: ROS/green_turtlebot3/urdf/green_turtlebot3.urdf.xacro (robot description, xacro)
@@ -4,11 +4,12 @@
     <xacro:include filename="$(find green_turtlebot3)/urdf/green_turtlebot3.gazebo.xacro"/>
     <xacro:property name="top_length" value="0.03"/>
-    <link name="base_footprint"/>
+    <xacro:property name="robot_name" value="green/"/>
+    <link name="${robot_name}base_footprint"/>
     <joint name="base_joint" type="fixed">
-        <parent link="base_footprint"/>
-        <child link="base_link"/>
+        <parent link="${robot_name}base_footprint"/>
+        <child link="${robot_name}base_link"/>
         <origin xyz="0 0 0.010" rpy="0 0 0"/>
     </joint>
-    <link name="base_link">
+    <link name="${robot_name}base_link">
         <visual>
             <origin xyz="-0.064 0 0.0" rpy="0 0 0"/>
@@ -33,53 +34,53 @@
         </inertial>
     </link>
-    <!--    add blue element   ********************** -->
-    <link name="stem">
-        <visual>
-            <origin xyz="0 0 0.0" rpy="0 0 0"/>
-            <geometry>
-                <cylinder length="0.1" radius="0.005"/>
-            </geometry>
-            <material name="dark"/>
-        </visual>
-        <collision>
-            <origin xyz="0 0 0" rpy="0 0 0"/>
-            <geometry>
-                <cylinder length="0.1" radius="0.005"/>
-            </geometry>
-        </collision>
-    </link>
-    <joint name="stem_joint" type="fixed">
-        <parent link="base_link"/>
-        <child link="stem"/>
-        <origin xyz="-0.16 0.07 0.14" rpy="0 0 0"/>
-    </joint>
-    <link name="top">
-        <visual>
-            <origin xyz="0 0 0.0" rpy="0 0 0"/>
-            <geometry>
-                <cylinder length="0.05" radius="0.05"/>
-            </geometry>
-            <material name="dark"/>
-        </visual>
-        <collision>
-            <origin xyz="0 0 0" rpy="0 0 0"/>
-            <geometry>
-                <cylinder length="${top_length}" radius="0.04"/>
-            </geometry>
-        </collision>
-    </link>
-    <joint name="top_joint" type="fixed">
-        <parent link="base_link"/>
-        <child link="top"/>
-        <origin xyz="-0.16 0.07 0.19" rpy="0 0 0"/>
-    </joint>
-    <!--    ************************************************-->
+    <!--    &lt;!&ndash;    add blue element   ********************** &ndash;&gt;-->
+    <!--    <link name="${robot_name}stem">-->
+    <!--        <visual>-->
+    <!--            <origin xyz="0 0 0.0" rpy="0 0 0"/>-->
+    <!--            <geometry>-->
+    <!--                <cylinder length="0.1" radius="0.005"/>-->
+    <!--            </geometry>-->
+    <!--            <material name="dark"/>-->
+    <!--        </visual>-->
+    <!--        <collision>-->
+    <!--            <origin xyz="0 0 0" rpy="0 0 0"/>-->
+    <!--            <geometry>-->
+    <!--                <cylinder length="0.1" radius="0.005"/>-->
+    <!--            </geometry>-->
+    <!--        </collision>-->
+    <!--    </link>-->
+    <!--    <joint name="stem_joint" type="fixed">-->
+    <!--        <parent link="${robot_name}base_link"/>-->
+    <!--        <child link="${robot_name}stem"/>-->
+    <!--        <origin xyz="-0.16 0.07 0.14" rpy="0 0 0"/>-->
+    <!--    </joint>-->
+    <!--    <link name="${robot_name}top">-->
+    <!--        <visual>-->
+    <!--            <origin xyz="0 0 0.0" rpy="0 0 0"/>-->
+    <!--            <geometry>-->
+    <!--                <cylinder length="0.05" radius="0.05"/>-->
+    <!--            </geometry>-->
+    <!--            <material name="dark"/>-->
+    <!--        </visual>-->
+    <!--        <collision>-->
+    <!--            <origin xyz="0 0 0" rpy="0 0 0"/>-->
+    <!--            <geometry>-->
+    <!--                <cylinder length="${top_length}" radius="0.04"/>-->
+    <!--            </geometry>-->
+    <!--        </collision>-->
+    <!--    </link>-->
+    <!--    <joint name="top_joint" type="fixed">-->
+    <!--        <parent link="${robot_name}base_link"/>-->
+    <!--        <child link="${robot_name}top"/>-->
+    <!--        <origin xyz="-0.16 0.07 0.19" rpy="0 0 0"/>-->
+    <!--    </joint>-->
+    <!--    &lt;!&ndash;    ************************************************&ndash;&gt;-->
     <joint name="wheel_left_joint" type="continuous">
-        <parent link="base_link"/>
-        <child link="wheel_left_link"/>
+        <parent link="${robot_name}base_link"/>
+        <child link="${robot_name}wheel_left_link"/>
         <origin xyz="0.0 0.144 0.023" rpy="-1.57 0 0"/>
         <axis xyz="0 0 1"/>
     </joint>
-    <link name="wheel_left_link">
+    <link name="${robot_name}wheel_left_link">
         <visual>
             <origin xyz="0 0 0" rpy="1.57 0 0"/>
@@ -105,10 +106,10 @@
     </link>
     <joint name="wheel_right_joint" type="continuous">
-        <parent link="base_link"/>
-        <child link="wheel_right_link"/>
+        <parent link="${robot_name}base_link"/>
+        <child link="${robot_name}wheel_right_link"/>
         <origin xyz="0.0 -0.144 0.023" rpy="-1.57 0 0"/>
         <axis xyz="0 0 1"/>
     </joint>
-    <link name="wheel_right_link">
+    <link name="${robot_name}wheel_right_link">
         <visual>
             <origin xyz="0 0 0" rpy="1.57 0 0"/>
@@ -134,9 +135,9 @@
     </link>
     <joint name="caster_back_right_joint" type="fixed">
-        <parent link="base_link"/>
-        <child link="caster_back_right_link"/>
+        <parent link="${robot_name}base_link"/>
+        <child link="${robot_name}caster_back_right_link"/>
         <origin xyz="-0.177 -0.064 -0.004" rpy="-1.57 0 0"/>
     </joint>
-    <link name="caster_back_right_link">
+    <link name="${robot_name}caster_back_right_link">
         <collision>
             <origin xyz="0 0.001 0" rpy="0 0 0"/>
@@ -154,9 +155,9 @@
     </link>
     <joint name="caster_back_left_joint" type="fixed">
-        <parent link="base_link"/>
-        <child link="caster_back_left_link"/>
+        <parent link="${robot_name}base_link"/>
+        <child link="${robot_name}caster_back_left_link"/>
         <origin xyz="-0.177 0.064 -0.004" rpy="-1.57 0 0"/>
     </joint>
-    <link name="caster_back_left_link">
+    <link name="${robot_name}caster_back_left_link">
         <collision>
             <origin xyz="0 0.001 0" rpy="0 0 0"/>
@@ -174,15 +175,15 @@
     </link>
     <joint name="imu_joint" type="fixed">
-        <parent link="base_link"/>
-        <child link="imu_link"/>
+        <parent link="${robot_name}base_link"/>
+        <child link="${robot_name}imu_link"/>
         <origin xyz="0.0 0 0.068" rpy="0 0 0"/>
     </joint>
-    <link name="imu_link"/>
+    <link name="${robot_name}imu_link"/>
     <joint name="scan_joint" type="fixed">
-        <parent link="base_link"/>
-        <child link="base_scan"/>
+        <parent link="${robot_name}base_link"/>
+        <child link="${robot_name}base_scan"/>
         <origin xyz="-0.064 0 0.122" rpy="0 0 0"/>
     </joint>
-    <link name="base_scan">
+    <link name="${robot_name}base_scan">
         <visual>
             <origin xyz="0 0 0.0" rpy="0 0 0"/>
@@ -208,8 +209,8 @@
     <joint name="camera_joint" type="fixed">
         <origin xyz="0.073 -0.011 0.084" rpy="0 0 0"/>
-        <parent link="base_link"/>
-        <child link="camera_link"/>
-    </joint>
-    <link name="camera_link">
+        <parent link="${robot_name}base_link"/>
+        <child link="${robot_name}camera_link"/>
+    </joint>
+    <link name="${robot_name}camera_link">
         <collision>
             <origin xyz="0.005 0.011 0.013" rpy="0 0 0"/>
@@ -221,13 +222,13 @@
     <joint name="camera_rgb_joint" type="fixed">
         <origin xyz="0.003 0.011 0.009" rpy="0 0 0"/>
-        <parent link="camera_link"/>
-        <child link="camera_rgb_frame"/>
-    </joint>
-    <link name="camera_rgb_frame"/>
+        <parent link="${robot_name}camera_link"/>
+        <child link="${robot_name}camera_rgb_frame"/>
+    </joint>
+    <link name="${robot_name}camera_rgb_frame"/>
     <joint name="camera_rgb_optical_joint" type="fixed">
         <origin xyz="0 0 0" rpy="-1.57 0 -1.57"/>
-        <parent link="camera_rgb_frame"/>
-        <child link="camera_rgb_optical_frame"/>
-    </joint>
-    <link name="camera_rgb_optical_frame"/>
+        <parent link="${robot_name}camera_rgb_frame"/>
+        <child link="${robot_name}camera_rgb_optical_frame"/>
+    </joint>
+    <link name="${robot_name}camera_rgb_optical_frame"/>
 </robot>

File: ROS/p_jfernandes/urdf/p_jfernandes.gazebo.xacro (robot description, xacro)
@@ -9,10 +9,10 @@
         <material>Gazebo/$(arg main_color)</material>
     </gazebo>
-    <gazebo reference="${robot_name}stem">
-        <material>Gazebo/$(arg main_color)</material>
-    </gazebo>
-    <gazebo reference="${robot_name}top">
-        <material>Gazebo/$(arg main_color)</material>
-    </gazebo>
+    <!--    <gazebo reference="${robot_name}stem">-->
+    <!--        <material>Gazebo/$(arg main_color)</material>-->
+    <!--    </gazebo>-->
+    <!--    <gazebo reference="${robot_name}top">-->
+    <!--        <material>Gazebo/$(arg main_color)</material>-->
+    <!--    </gazebo>-->
     <gazebo reference="${robot_name}wheel_left_link">
         <mu1>0.1</mu1>
@@ -67,4 +67,5 @@
             <odometrySource>world</odometrySource>
             <publishOdomTF>true</publishOdomTF>
+            <!--            <publishOdomTF>false</publishOdomTF>-->
             <robotBaseFrame>${robot_name}base_footprint</robotBaseFrame>
             <publishWheelTF>false</publishWheelTF>

File: ROS/p_jfernandes/urdf/p_jfernandes.urdf.xacro (robot description, xacro)
@@ -34,46 +34,46 @@
         </inertial>
     </link>
-    <!--    add blue element   ********************** -->
-    <link name="${robot_name}stem">
-        <visual>
-            <origin xyz="0 0 0.0" rpy="0 0 0"/>
-            <geometry>
-                <cylinder length="0.1" radius="0.005"/>
-            </geometry>
-            <material name="dark"/>
-        </visual>
-        <collision>
-            <origin xyz="0 0 0" rpy="0 0 0"/>
-            <geometry>
-                <cylinder length="0.1" radius="0.005"/>
-            </geometry>
-        </collision>
-    </link>
-    <joint name="stem_joint" type="fixed">
-        <parent link="${robot_name}base_link"/>
-        <child link="${robot_name}stem"/>
-        <origin xyz="-0.16 0.07 0.14" rpy="0 0 0"/>
-    </joint>
-    <link name="${robot_name}top">
-        <visual>
-            <origin xyz="0 0 0.0" rpy="0 0 0"/>
-            <geometry>
-                <cylinder length="0.05" radius="0.05"/>
-            </geometry>
-            <material name="dark"/>
-        </visual>
-        <collision>
-            <origin xyz="0 0 0" rpy="0 0 0"/>
-            <geometry>
-                <cylinder length="${top_length}" radius="0.04"/>
-            </geometry>
-        </collision>
-    </link>
-    <joint name="top_joint" type="fixed">
-        <parent link="${robot_name}base_link"/>
-        <child link="${robot_name}top"/>
-        <origin xyz="-0.16 0.07 0.19" rpy="0 0 0"/>
-    </joint>
-    <!--    ************************************************-->
+<!--    &lt;!&ndash;    add blue element   ********************** &ndash;&gt;-->
+<!--    <link name="${robot_name}stem">-->
+<!--        <visual>-->
+<!--            <origin xyz="0 0 0.0" rpy="0 0 0"/>-->
+<!--            <geometry>-->
+<!--                <cylinder length="0.1" radius="0.005"/>-->
+<!--            </geometry>-->
+<!--            <material name="dark"/>-->
+<!--        </visual>-->
+<!--        <collision>-->
+<!--            <origin xyz="0 0 0" rpy="0 0 0"/>-->
+<!--            <geometry>-->
+<!--                <cylinder length="0.1" radius="0.005"/>-->
+<!--            </geometry>-->
+<!--        </collision>-->
+<!--    </link>-->
+<!--    <joint name="stem_joint" type="fixed">-->
+<!--        <parent link="${robot_name}base_link"/>-->
+<!--        <child link="${robot_name}stem"/>-->
+<!--        <origin xyz="-0.16 0.07 0.14" rpy="0 0 0"/>-->
+<!--    </joint>-->
+<!--    <link name="${robot_name}top">-->
+<!--        <visual>-->
+<!--            <origin xyz="0 0 0.0" rpy="0 0 0"/>-->
+<!--            <geometry>-->
+<!--                <cylinder length="0.05" radius="0.05"/>-->
+<!--            </geometry>-->
+<!--            <material name="dark"/>-->
+<!--        </visual>-->
+<!--        <collision>-->
+<!--            <origin xyz="0 0 0" rpy="0 0 0"/>-->
+<!--            <geometry>-->
+<!--                <cylinder length="${top_length}" radius="0.04"/>-->
+<!--            </geometry>-->
+<!--        </collision>-->
+<!--    </link>-->
+<!--    <joint name="top_joint" type="fixed">-->
+<!--        <parent link="${robot_name}base_link"/>-->
+<!--        <child link="${robot_name}top"/>-->
+<!--        <origin xyz="-0.16 0.07 0.19" rpy="0 0 0"/>-->
+<!--    </joint>-->
+<!--    &lt;!&ndash;    ************************************************&ndash;&gt;-->
     <joint name="wheel_left_joint" type="continuous">
         <parent link="${robot_name}base_link"/>
