Commit message: update

File: ROS/p_jfernandes_v2.0/p_jfernandes_description/urdf/p_jfernandes.urdf.xacro (robot description, xacro)
@@ -1,15 +1,18 @@
 <?xml version="1.0" ?>
-<robot name="p_jfernandes" xmlns:xacro="http://ros.org/wiki/xacro">
-    <xacro:include filename="$(find turtlebot3_description)/urdf/common_properties.xacro"/>
-    <xacro:include filename="$(find p_jfernandes)/urdf/p_jfernandes.gazebo.xacro"/>
+<robot name="team_hunt_player" xmlns:xacro="http://ros.org/wiki/xacro">
+    <xacro:arg name="player_name" default="p_jfernandes"/>
+    <xacro:arg name="player_color" default="Blue"/>
+    <xacro:property name="player_name" value="$(arg player_name)"/>
+    <xacro:property name="player_color" value="$(arg player_color)"/>
     <xacro:property name="top_length" value="0.03"/>
-    <xacro:property name="robot_name" value="p_jfernandes/"/>
-    <link name="${robot_name}base_footprint"/>
+    <xacro:include filename="$(find p_jfernandes_description)/urdf/properties.xacro"/>
+    <xacro:include filename="$(find p_jfernandes_description)/urdf/p_jfernandes.gazebo.xacro"/>
+    <link name="base_footprint"/>
     <joint name="base_joint" type="fixed">
-        <parent link="${robot_name}base_footprint"/>
-        <child link="${robot_name}base_link"/>
+        <parent link="base_footprint"/>
+        <child link="base_link"/>
         <origin xyz="0 0 0.010" rpy="0 0 0"/>
     </joint>
-    <link name="${robot_name}base_link">
+    <link name="base_link">
         <visual>
             <origin xyz="-0.064 0 0.0" rpy="0 0 0"/>
@@ -18,5 +21,5 @@
                       scale="0.001 0.001 0.001"/>
             </geometry>
-            <material name="light_black"/>
+            <material name="$(arg player_color)"/>
         </visual>
         <collision>
@@ -35,5 +38,5 @@
     </link>
     <!--    &lt;!&ndash;    add blue element   ********************** &ndash;&gt;-->
-    <!--    <link name="${robot_name}stem">-->
+    <!--    <link name="stem">-->
     <!--        <visual>-->
     <!--            <origin xyz="0 0 0.0" rpy="0 0 0"/>-->
@@ -51,9 +54,9 @@
     <!--    </link>-->
     <!--    <joint name="stem_joint" type="fixed">-->
-    <!--        <parent link="${robot_name}base_link"/>-->
-    <!--        <child link="${robot_name}stem"/>-->
+    <!--        <parent link="base_link"/>-->
+    <!--        <child link="stem"/>-->
     <!--        <origin xyz="-0.16 0.07 0.14" rpy="0 0 0"/>-->
     <!--    </joint>-->
-    <!--    <link name="${robot_name}top">-->
+    <!--    <link name="top">-->
     <!--        <visual>-->
     <!--            <origin xyz="0 0 0.0" rpy="0 0 0"/>-->
@@ -71,16 +74,16 @@
     <!--    </link>-->
     <!--    <joint name="top_joint" type="fixed">-->
-    <!--        <parent link="${robot_name}base_link"/>-->
-    <!--        <child link="${robot_name}top"/>-->
+    <!--        <parent link="base_link"/>-->
+    <!--        <child link="top"/>-->
     <!--        <origin xyz="-0.16 0.07 0.19" rpy="0 0 0"/>-->
     <!--    </joint>-->
     <!--    &lt;!&ndash;    ************************************************&ndash;&gt;-->
     <joint name="wheel_left_joint" type="continuous">
-        <parent link="${robot_name}base_link"/>
-        <child link="${robot_name}wheel_left_link"/>
+        <parent link="base_link"/>
+        <child link="wheel_left_link"/>
         <origin xyz="0.0 0.144 0.023" rpy="-1.57 0 0"/>
         <axis xyz="0 0 1"/>
     </joint>
-    <link name="${robot_name}wheel_left_link">
+    <link name="wheel_left_link">
         <visual>
             <origin xyz="0 0 0" rpy="1.57 0 0"/>
@@ -106,10 +109,10 @@
     </link>
     <joint name="wheel_right_joint" type="continuous">
-        <parent link="${robot_name}base_link"/>
-        <child link="${robot_name}wheel_right_link"/>
+        <parent link="base_link"/>
+        <child link="wheel_right_link"/>
         <origin xyz="0.0 -0.144 0.023" rpy="-1.57 0 0"/>
         <axis xyz="0 0 1"/>
     </joint>
-    <link name="${robot_name}wheel_right_link">
+    <link name="wheel_right_link">
         <visual>
             <origin xyz="0 0 0" rpy="1.57 0 0"/>
@@ -135,9 +138,9 @@
     </link>
     <joint name="caster_back_right_joint" type="fixed">
-        <parent link="${robot_name}base_link"/>
-        <child link="${robot_name}caster_back_right_link"/>
+        <parent link="base_link"/>
+        <child link="caster_back_right_link"/>
         <origin xyz="-0.177 -0.064 -0.004" rpy="-1.57 0 0"/>
     </joint>
-    <link name="${robot_name}caster_back_right_link">
+    <link name="caster_back_right_link">
         <collision>
             <origin xyz="0 0.001 0" rpy="0 0 0"/>
@@ -155,9 +158,9 @@
     </link>
     <joint name="caster_back_left_joint" type="fixed">
-        <parent link="${robot_name}base_link"/>
-        <child link="${robot_name}caster_back_left_link"/>
+        <parent link="base_link"/>
+        <child link="caster_back_left_link"/>
         <origin xyz="-0.177 0.064 -0.004" rpy="-1.57 0 0"/>
     </joint>
-    <link name="${robot_name}caster_back_left_link">
+    <link name="caster_back_left_link">
         <collision>
             <origin xyz="0 0.001 0" rpy="0 0 0"/>
@@ -175,15 +178,15 @@
     </link>
     <joint name="imu_joint" type="fixed">
-        <parent link="${robot_name}base_link"/>
-        <child link="${robot_name}imu_link"/>
+        <parent link="base_link"/>
+        <child link="imu_link"/>
         <origin xyz="0.0 0 0.068" rpy="0 0 0"/>
     </joint>
-    <link name="${robot_name}imu_link"/>
+    <link name="imu_link"/>
     <joint name="scan_joint" type="fixed">
-        <parent link="${robot_name}base_link"/>
-        <child link="${robot_name}base_scan"/>
+        <parent link="base_link"/>
+        <child link="base_scan"/>
         <origin xyz="-0.064 0 0.122" rpy="0 0 0"/>
     </joint>
-    <link name="${robot_name}base_scan">
+    <link name="base_scan">
         <visual>
             <origin xyz="0 0 0.0" rpy="0 0 0"/>
@@ -209,8 +212,8 @@
     <joint name="camera_joint" type="fixed">
         <origin xyz="0.073 -0.011 0.084" rpy="0 0 0"/>
-        <parent link="${robot_name}base_link"/>
-        <child link="${robot_name}camera_link"/>
-    </joint>
-    <link name="${robot_name}camera_link">
+        <parent link="base_link"/>
+        <child link="camera_link"/>
+    </joint>
+    <link name="camera_link">
         <collision>
             <origin xyz="0.005 0.011 0.013" rpy="0 0 0"/>
@@ -222,13 +225,13 @@
     <joint name="camera_rgb_joint" type="fixed">
         <origin xyz="0.003 0.011 0.009" rpy="0 0 0"/>
-        <parent link="${robot_name}camera_link"/>
-        <child link="${robot_name}camera_rgb_frame"/>
-    </joint>
-    <link name="${robot_name}camera_rgb_frame"/>
+        <parent link="camera_link"/>
+        <child link="camera_rgb_frame"/>
+    </joint>
+    <link name="camera_rgb_frame"/>
     <joint name="camera_rgb_optical_joint" type="fixed">
         <origin xyz="0 0 0" rpy="-1.57 0 -1.57"/>
-        <parent link="${robot_name}camera_rgb_frame"/>
-        <child link="${robot_name}camera_rgb_optical_frame"/>
-    </joint>
-    <link name="${robot_name}camera_rgb_optical_frame"/>
+        <parent link="camera_rgb_frame"/>
+        <child link="camera_rgb_optical_frame"/>
+    </joint>
+    <link name="camera_rgb_optical_frame"/>
 </robot>

Commit message: update

File: ROS/p_jfernandes_v2.0/p_jfernandes_description/urdf/p_jfernandes.urdf.xacro (robot description, xacro)
@@ -90,5 +90,5 @@
             <origin xyz="0 0 0" rpy="0 0 0"/>
             <geometry>
-                <box size="0.05 0.1 0.001"/>
+                <box size="0.05 0.05 0.001"/>
             </geometry>
         </collision>

Commit message: update

File: ROS/p_jfernandes_v2.0/p_jfernandes_description/urdf/p_jfernandes.urdf.xacro (robot description, xacro)
@@ -49,5 +49,5 @@
             <origin xyz="0 0 0" rpy="0 0 0"/>
             <geometry>
-                <cylinder length="0.07" radius="0.002"/>
+                <cylinder length="0" radius="0"/>
             </geometry>
         </collision>
@@ -69,5 +69,5 @@
             <origin xyz="0 0 0" rpy="0 0 0"/>
             <geometry>
-                <cylinder length="0.07" radius="0.002"/>
+                <cylinder length="0" radius="0"/>
             </geometry>
         </collision>
@@ -90,5 +90,5 @@
             <origin xyz="0 0 0" rpy="0 0 0"/>
             <geometry>
-                <box size="0.05 0.05 0.001"/>
+                <box size="0 0 0"/>
             </geometry>
         </collision>

Commit message: update

File: ROS/p_jfernandes_v2.0/p_jfernandes_description/urdf/p_jfernandes.urdf.xacro (robot description, xacro)
@@ -46,10 +46,10 @@
             <material name="dark"/>
         </visual>
-        <collision>
-            <origin xyz="0 0 0" rpy="0 0 0"/>
-            <geometry>
-                <cylinder length="0" radius="0"/>
-            </geometry>
-        </collision>
+        <!--        <collision>-->
+        <!--            <origin xyz="0 0 0" rpy="0 0 0"/>-->
+        <!--            <geometry>-->
+        <!--                <cylinder length="0" radius="0"/>-->
+        <!--            </geometry>-->
+        <!--        </collision>-->
     </link>
     <joint name="stem_left_joint" type="fixed">
@@ -66,10 +66,10 @@
             <material name="dark"/>
         </visual>
-        <collision>
-            <origin xyz="0 0 0" rpy="0 0 0"/>
-            <geometry>
-                <cylinder length="0" radius="0"/>
-            </geometry>
-        </collision>
+        <!--        <collision>-->
+        <!--            <origin xyz="0 0 0" rpy="0 0 0"/>-->
+        <!--            <geometry>-->
+        <!--                <cylinder length="0" radius="0"/>-->
+        <!--            </geometry>-->
+        <!--        </collision>-->
     </link>
     <joint name="stem_right_joint" type="fixed">
@@ -87,10 +87,10 @@
             <material name="dark"/>
         </visual>
-        <collision>
-            <origin xyz="0 0 0" rpy="0 0 0"/>
-            <geometry>
-                <box size="0 0 0"/>
-            </geometry>
-        </collision>
+        <!--        <collision>-->
+        <!--            <origin xyz="0 0 0" rpy="0 0 0"/>-->
+        <!--            <geometry>-->
+        <!--                <box size="0 0 0"/>-->
+        <!--            </geometry>-->
+        <!--        </collision>-->
     </link>
     <joint name="spoiler_joint" type="fixed">
@@ -100,4 +100,5 @@
         <!--                <origin xyz="-0.16 -0.43 0.16" rpy="0 0.5 0"/>-->
     </joint>
+    <!--    ************************************************-->
     <!--    <link name="top">-->
     <!--        <visual>-->
@@ -120,5 +121,5 @@
     <!--        <origin xyz="-0.16 0.07 0.19" rpy="0 0 0"/>-->
     <!--    </joint>-->
-    <!--    &lt;!&ndash;    ************************************************&ndash;&gt;-->
+    <!--    ************************************************-->
     <joint name="wheel_left_joint" type="continuous">
         <parent link="base_link"/>
