Commit message: update

File: ROS/p_jfernandes_v2.0/p_jfernandes_description/urdf/p_jfernandes.gazebo.xacro (robot description, xacro)
@@ -7,10 +7,13 @@
         <material>Gazebo/${player_color}</material>
     </gazebo>
-    <!--    <gazebo reference="stem">-->
-    <!--        <material>Gazebo/$(arg main_color)</material>-->
-    <!--    </gazebo>-->
-    <!--    <gazebo reference="top">-->
-    <!--        <material>Gazebo/$(arg main_color)</material>-->
-    <!--    </gazebo>-->
+    <gazebo reference="stem_left">
+        <material>Gazebo/DarkGrey</material>
+    </gazebo>
+    <gazebo reference="stem_right">
+        <material>Gazebo/DarkGrey</material>
+    </gazebo>
+    <gazebo reference="spoiler">
+        <material>Gazebo/DarkGrey</material>
+    </gazebo>
     <gazebo reference="wheel_left_link">
         <mu1>0.1</mu1>
@@ -21,5 +24,5 @@
         <maxVel>0.1</maxVel>
         <fdir1>1 0 0</fdir1>
-        <material>Gazebo/FlatBlack</material>
+        <material>Gazebo/DarkGrey</material>
     </gazebo>
     <gazebo reference="wheel_right_link">
@@ -31,5 +34,5 @@
         <maxVel>0.1</maxVel>
         <fdir1>1 0 0</fdir1>
-        <material>Gazebo/FlatBlack</material>
+        <material>Gazebo/DarkGrey</material>
     </gazebo>
     <gazebo reference="caster_back_right_link">
@@ -111,5 +114,5 @@
     </gazebo>
     <gazebo reference="base_scan">
-        <material>Gazebo/FlatBlack</material>
+        <material>Gazebo/DarkGrey</material>
         <sensor type="ray" name="lds_lfcd_sensor">
             <pose>0 0 0 0 0 0</pose>

File: ROS/p_jfernandes_v2.0/p_jfernandes_description/urdf/p_jfernandes.urdf.xacro (robot description, xacro)
@@ -37,25 +37,67 @@
         </inertial>
     </link>
-    <!--    &lt;!&ndash;    add blue element   ********************** &ndash;&gt;-->
-    <!--    <link name="stem">-->
-    <!--        <visual>-->
-    <!--            <origin xyz="0 0 0.0" rpy="0 0 0"/>-->
-    <!--            <geometry>-->
-    <!--                <cylinder length="0.1" radius="0.005"/>-->
-    <!--            </geometry>-->
-    <!--            <material name="dark"/>-->
-    <!--        </visual>-->
-    <!--        <collision>-->
-    <!--            <origin xyz="0 0 0" rpy="0 0 0"/>-->
-    <!--            <geometry>-->
-    <!--                <cylinder length="0.1" radius="0.005"/>-->
-    <!--            </geometry>-->
-    <!--        </collision>-->
-    <!--    </link>-->
-    <!--    <joint name="stem_joint" type="fixed">-->
-    <!--        <parent link="base_link"/>-->
-    <!--        <child link="stem"/>-->
-    <!--        <origin xyz="-0.16 0.07 0.14" rpy="0 0 0"/>-->
-    <!--    </joint>-->
+    <!--    add blue element   ********************** -->
+    <link name="stem_left">
+        <visual>
+            <origin xyz="0 0 0.0" rpy="0 0 0"/>
+            <geometry>
+                <cylinder length="0.07" radius="0.002"/>
+            </geometry>
+            <material name="dark"/>
+        </visual>
+        <collision>
+            <origin xyz="0 0 0" rpy="0 0 0"/>
+            <geometry>
+                <cylinder length="0.07" radius="0.002"/>
+            </geometry>
+        </collision>
+    </link>
+    <joint name="stem_left_joint" type="fixed">
+        <parent link="base_link"/>
+        <child link="stem_left"/>
+        <origin xyz="-0.18 0.07 0.12" rpy="0 0 0"/>
+    </joint>
+    <link name="stem_right">
+        <visual>
+            <origin xyz="0 0 0.0" rpy="0 0 0"/>
+            <geometry>
+                <cylinder length="0.07" radius="0.002"/>
+            </geometry>
+            <material name="dark"/>
+        </visual>
+        <collision>
+            <origin xyz="0 0 0" rpy="0 0 0"/>
+            <geometry>
+                <cylinder length="0.07" radius="0.002"/>
+            </geometry>
+        </collision>
+    </link>
+    <joint name="stem_right_joint" type="fixed">
+        <parent link="base_link"/>
+        <child link="stem_right"/>
+        <origin xyz="-0.18 -0.07 0.12" rpy="0 0 0"/>
+    </joint>
+    <link name="spoiler">
+        <visual>
+            <origin xyz="0 0 0.0" rpy="0 0 0"/>
+            <geometry>
+                <!--                <box size="0.07 0.2 0.001"/>-->
+                <mesh filename="package://p_jfernandes_description/meshes/spoiler.dae" scale="0.005 0.005 0.005"/>
+            </geometry>
+            <material name="dark"/>
+        </visual>
+        <collision>
+            <origin xyz="0 0 0" rpy="0 0 0"/>
+            <geometry>
+                <box size="0.07 0.2 0.001"/>
+            </geometry>
+        </collision>
+    </link>
+    <joint name="spoiler_joint" type="fixed">
+        <parent link="base_link"/>
+        <child link="spoiler"/>
+        <origin xyz="-0.38 -0.46 0.01" rpy="0 0.5 0"/>
+        <!--                <origin xyz="-0.16 -0.43 0.16" rpy="0 0.5 0"/>-->
+    </joint>
     <!--    <link name="top">-->
     <!--        <visual>-->

Commit message: update

File: ROS/p_jfernandes_v2.0/p_jfernandes_description/urdf/p_jfernandes.gazebo.xacro (robot description, xacro)
@@ -122,4 +122,5 @@
                 <scan>
                     <horizontal>
+                        <!--                        number of lidar points per rotation, here = 360-->
                         <samples>360</samples>
                         <resolution>1</resolution>
@@ -155,6 +156,6 @@
                     <!--                    <width>640</width>-->
                     <!--                    <height>480</height>-->
-                    <width>1000</width>
-                    <height>800</height>
+                    <width>1200</width>
+                    <height>600</height>
                     <format>R8G8B8</format>
                 </image>

File: ROS/p_jfernandes_v2.0/p_jfernandes_description/urdf/p_jfernandes.urdf.xacro (robot description, xacro)
@@ -90,5 +90,5 @@
             <origin xyz="0 0 0" rpy="0 0 0"/>
             <geometry>
-                <box size="0.07 0.2 0.001"/>
+                <box size="0.05 0.1 0.001"/>
             </geometry>
         </collision>

Commit message: update

File: ROS/p_jfernandes_v2.0/p_jfernandes_description/urdf/p_jfernandes.gazebo.xacro (robot description, xacro)
@@ -15,4 +15,18 @@
     <gazebo reference="spoiler">
         <material>Gazebo/DarkGrey</material>
+    </gazebo>
+    <!--    bumper sensor-->
+    <gazebo reference="base_link">
+        <sensor name="base_link" type="contact">
+            <update_rate>1000.0</update_rate>
+            <always_on>true</always_on>
+            <contact>
+                <collision>base_footprint_fixed_joint_lump__base_link_collision</collision>
+            </contact>
+            <plugin name="base_link_contact_sensor_plugin" filename="libgazebo_ros_bumper.so">
+                <bumperTopicName>contact</bumperTopicName>
+                <frameName>world</frameName>
+            </plugin>
+        </sensor>
     </gazebo>
     <gazebo reference="wheel_left_link">
